File: circuit_files/Kallebol_elevation.kicad_pcb (KiCad board)
At the start: 2 copper layers, 86.9 x 80.3 mm, 38 parts, among them J1 Limit_switch, J2 Home_switch, J3 UART_conn, J4 Power in, J5 power_out, J6 Programming header, J7 Encoder, U1 DMC3021LSD, U2 DMC3021LSD, U3 PIC16F874-PLCC44, U4 LM7805_TO220, U5 DMC3021LSD, Y1 Crystal_Small

Commit message: layout done
Parts:
- removed U3: PIC16F874-PLCC44, Package_LCC:PLCC-44
- removed U4: LM7805_TO220, Package_TO_SOT_THT:TO-220-3_Vertical
- removed U5: DMC3021LSD, Package_SO:SOIC-8_3.9x4.9mm_P1.27mm
- removed Y1: Crystal_Small, Crystal:Crystal_HC18-U_Vertical
- added C10: 100nF, Capacitor_SMD:C_0603_1608Metric_Pad1.08x0.95mm_HandSolder, F.Cu at (107.5, 61.2)
- added C11: C_Small, Capacitor_SMD:C_0603_1608Metric_Pad1.08x0.95mm_HandSolder, F.Cu at (84.1, 117.4)
- added C12: 4.7µF, Capacitor_SMD:CP_Elec_10x10, F.Cu at (78.2, 109.2)
- added C13: 4.7µF, Capacitor_SMD:CP_Elec_10x10, F.Cu at (78.5, 85.3)
- added C9: 1uF, Capacitor_SMD:C_0603_1608Metric_Pad1.08x0.95mm_HandSolder, F.Cu at (104.7, 63.2)
- added D4: LED, LED_SMD:LED_0603_1608Metric, F.Cu at (121.7, 86.4)
- added D5: LED, LED_SMD:LED_0603_1608Metric, F.Cu at (121.7, 84.6)
- added IC1: BD62130AEFJ-E2, Motor_drv:SOIC127P600X100-9N, F.Cu at (65.0, 74.9)
- added J10: Conn_01x05_Male, Connector_PinSocket_2.54mm:PinSocket_1x05_P2.54mm_Vertical, F.Cu at (87.1, 78.2)
- added J11: UART/I2C, Connector_PinSocket_2.54mm:PinSocket_1x03_P2.54mm_Vertical, F.Cu at (122.7, 122.4)
- added J8: RF_switch, Connector_PinSocket_2.54mm:PinSocket_1x10_P2.54mm_Vertical, F.Cu at (131.8, 112.8)
- added J9: Conn_01x05_Male, Connector_PinSocket_2.54mm:PinSocket_1x05_P2.54mm_Vertical, F.Cu at (86.9, 93.2)
- added JP1: Jumper_3, Connector_PinSocket_2.54mm:PinSocket_1x03_P2.54mm_Vertical, F.Cu at (86.9, 106.9)
- added Q1: BUK9880, Package_TO_SOT_SMD:SOT-223-3_TabPin2, F.Cu at (123.4, 103.6)
- added Q2: BUK9880, Package_TO_SOT_SMD:SOT-223-3_TabPin2, F.Cu at (123.4, 93.5)
- added R10: 10k, Resistor_SMD:R_0603_1608Metric_Pad0.98x0.95mm_HandSolder, F.Cu at (69.7, 58.7)
- added R11: 10k, Resistor_SMD:R_0603_1608Metric_Pad0.98x0.95mm_HandSolder, F.Cu at (107.5, 58.7)
- added R12: 10k, Resistor_SMD:R_0603_1608Metric_Pad0.98x0.95mm_HandSolder, F.Cu at (87.3, 60.7)
- added R13: 10k, Resistor_SMD:R_0603_1608Metric_Pad0.98x0.95mm_HandSolder, F.Cu at (99.2, 58.9)
- added R14: 550, Resistor_SMD:R_0603_1608Metric_Pad0.98x0.95mm_HandSolder, F.Cu at (121.5, 73.4)
- added R15: 550, Resistor_SMD:R_0603_1608Metric_Pad0.98x0.95mm_HandSolder, F.Cu at (121.5, 75.2)
- C1: value 22p -> 4.7µF; footprint Capacitor_SMD:C_0603_1608Metric_Pad1.05x0.95mm_HandSolder -> Capacitor_SMD:CP_Elec_10x10
- C2: value 22p -> 1µF; footprint Capacitor_SMD:C_0603_1608Metric_Pad1.05x0.95mm_HandSolder -> Capacitor_SMD:C_0603_1608Metric_Pad1.08x0.95mm_HandSolder
- C3, C4, C7: value C_power -> 100nF; footprint Capacitor_THT:CP_Radial_D10.0mm_P5.00mm -> Capacitor_SMD:C_0603_1608Metric_Pad1.08x0.95mm_HandSolder
- C5: value C_Small -> 4.7µF; footprint Capacitor_SMD:C_0603_1608Metric_Pad1.05x0.95mm_HandSolder -> Capacitor_SMD:CP_Elec_10x10
- C6: value C_Small -> 100nF; footprint Capacitor_SMD:C_0603_1608Metric_Pad1.05x0.95mm_HandSolder -> Capacitor_SMD:C_0603_1608Metric_Pad1.08x0.95mm_HandSolder
- C8: footprint Capacitor_SMD:C_0603_1608Metric_Pad1.05x0.95mm_HandSolder -> Capacitor_SMD:C_0603_1608Metric_Pad1.08x0.95mm_HandSolder
- F1: footprint Xp_motor:Fuse_holder -> Fuse:Fuseholder_Cylinder-5x20mm_Wuerth_696103101002-SMD_Horizontal_Open
- J1: value Limit_switch -> Home_switch; footprint TerminalBlock:TerminalBlock_bornier-2_P5.08mm -> TerminalBlock_Phoenix:TerminalBlock_Phoenix_MKDS-1,5-3_1x03_P5.00mm_Horizontal
- J2: value Home_switch -> Encoder; footprint TerminalBlock:TerminalBlock_bornier-2_P5.08mm -> TerminalBlock_Phoenix:TerminalBlock_Phoenix_MKDS-1,5-3_1x03_P5.00mm_Horizontal
- J3: value UART_conn -> Limit Switch; footprint TerminalBlock:TerminalBlock_bornier-2_P5.08mm -> TerminalBlock_Phoenix:TerminalBlock_Phoenix_MKDS-1,5-3_1x03_P5.00mm_Horizontal
- J6: value Programming header -> Screw_Terminal_01x02; footprint Connector_PinSocket_2.54mm:PinSocket_1x06_P2.54mm_Vertical -> TerminalBlock:TerminalBlock_bornier-2_P5.08mm
- J7: value Encoder -> Screw_Terminal_01x02; footprint Connector_PinSocket_2.54mm:PinSocket_1x03_P2.54mm_Vertical -> TerminalBlock:TerminalBlock_bornier-2_P5.08mm
- R1, R2: value 10k -> 26k; footprint Resistor_SMD:R_0603_1608Metric_Pad1.05x0.95mm_HandSolder -> Resistor_SMD:R_0603_1608Metric_Pad0.98x0.95mm_HandSolder
- R3, R4: value 10k -> 40k; footprint Resistor_SMD:R_0603_1608Metric_Pad1.05x0.95mm_HandSolder -> Resistor_SMD:R_0603_1608Metric_Pad0.98x0.95mm_HandSolder
- R5, R6, R8, R9: footprint Resistor_SMD:R_0603_1608Metric_Pad1.05x0.95mm_HandSolder -> Resistor_SMD:R_0603_1608Metric_Pad0.98x0.95mm_HandSolder
- R7: value 30k -> 10k; footprint Resistor_SMD:R_0603_1608Metric_Pad1.05x0.95mm_HandSolder -> Resistor_SMD:R_0603_1608Metric_Pad0.98x0.95mm_HandSolder
- U1: value DMC3021LSD -> L7805; footprint Package_SO:SOIC-8_3.9x4.9mm_P1.27mm -> Package_TO_SOT_SMD:SOT-223-3_TabPin2
- U2: value DMC3021LSD -> Pico; footprint Package_SO:SOIC-8_3.9x4.9mm_P1.27mm -> MCU_RaspberryPi_and_Boards:RPi_Pico_SMD_TH
- moved R2 72.1 mm to (64.9, 60.7), turned to 0 degrees
- moved R7 61.9 mm to (87.3, 58.7), turned to 0 degrees
- moved C2 61.0 mm to (59.6, 80.5), turned to 180 degrees
- moved C1 54.1 mm to (66.8, 85.3), turned to 90 degrees
- moved C5 54.0 mm to (78.2, 98.0)
- moved J6 51.1 mm to (131.1, 76.2)
- moved C8 50.6 mm to (86.4, 117.5), turned to 90 degrees
- moved C7 46.5 mm to (74.3, 60.7), turned to 180 degrees
- moved R9 41.9 mm to (69.7, 60.7), turned to 180 degrees
- moved J1 38.7 mm to (81.3, 51.1)
- moved J5 38.0 mm to (52.8, 75.2), turned to 90 degrees
- moved C4 37.4 mm to (91.8, 60.7), turned to 180 degrees
- moved U1 36.9 mm to (79.0, 120.7)
- moved J4 36.4 mm to (53.1, 104.6), turned to -90 degrees
- moved R5 34.7 mm to (121.5, 77.0), turned to 180 degrees
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Connections:
- C1 pad 1: Net-(C1-Pad1) -> +12V
- C2 pad 1: Net-(C2-Pad1) -> +12V
- C4 pad 1: +12V -> GND
- C4 pad 2: GND -> Home
- C5 pad 1: Enc_2 -> +12V
- C5 pad 2: +5V -> GND
- C6 pad 2: +5V -> GND
- C7 pad 1: +5V -> GND
- C7 pad 2: GND -> Limit
- D1 pad 2: Net-(D1-Pad2) -> Net-(D1-A)
- D3 pad 2: Net-(D3-Pad2) -> Net-(D3-A)
- F1 pad 2: Net-(F1-Pad2) -> +12V
- J1 pad 1: Limit -> +12V
- J1 pad 2: +5V -> Net-(J1-Pin_2)
- J2 pad 1: Home -> Net-(J2-Pin_1)
- J2 pad 2: +5V -> +3V3
- J3 pad 1: UART_RX -> +12V
- J3 pad 2: UART_TX -> Net-(J3-Pin_2)
- J6 pad 1: MCLR -> Net-(J6-Pin_1)
- J6 pad 2: +5V -> +12V
- J7 pad 1: Enc_2 -> Net-(J7-Pin_1)
- J7 pad 2: GND -> +12V
- R1 pad 1: Home -> +12V
- R1 pad 2: GND -> Net-(J1-Pin_2)
- R2 pad 1: MCLR -> +12V
- R2 pad 2: +5V -> Net-(J3-Pin_2)
- R3 pad 1: Enc_2 -> Load1_enable
- R3 pad 2: +5V -> GND
- R4 pad 1: Enc_1 -> Load2_enable
- R4 pad 2: +5V -> GND
- R7 pad 1: Net-(R7-Pad1) -> Net-(J1-Pin_2)
- R9 pad 2: GND -> Net-(J3-Pin_2)
- U1 pad 1: GND -> +12V
- U1 pad 2: Hb1 -> GND
- U1 pad 3: +12V -> +5V
- U2 pad 1: GND -> Net-(J11-Pin_1)
- U2 pad 2: Hb2 -> Net-(J11-Pin_2)
- U2 pad 3: +12V -> GND
- U2 pad 4: Hb2 -> Net-(J8-Pin_1)
- U2 pad 5: P_out2 -> Net-(J8-Pin_2)
- U2 pad 6: P_out2 -> Net-(J8-Pin_3)
- U2 pad 7: P_out2 -> Net-(J8-Pin_4)
- U2 pad 8: P_out2 -> GND
Routing:
- net +12V: track 79.0 -> 236.0 mm, vias 0 -> 3
- net +5V: track 174.0 -> 59.8 mm, vias 2 -> 0
- net +3V3: track 0.00 -> 78.0 mm, vias 0 -> 2
- net UART_RX: track 38.3 -> 0.00 mm, vias 2 -> 0
- net UART_TX: track 38.0 -> 0.00 mm, vias 2 -> 0
- net Net-(J7-Pin_1): track 0.00 -> 35.9 mm
- net Net-(J6-Pin_1): track 0.00 -> 32.9 mm
- net Net-(J8-Pin_4): track 0.00 -> 25.9 mm
- net Net-(J8-Pin_3): track 0.00 -> 23.7 mm
- net Net-(J8-Pin_2): track 0.00 -> 21.7 mm
- net Load1_enable: track 0.00 -> 20.7 mm
- net Net-(J8-Pin_1): track 0.00 -> 20.4 mm
- net Enc_1: track 64.3 -> 46.7 mm
- net Limit: track 34.1 -> 50.5 mm
- net Net-(D4-K): track 0.00 -> 16.1 mm
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Other:
- net class Chonk removed
- net class Default removed
- board text added: "+12v - GND"
- board text added: "Skrot AB SA6DGJ 2023-03-29 Elevation controll v2"
- board text removed: "12VDC - GND"
- board text removed: "Encoder I/O-5v-I/O"
- board text removed: "Home Switch I/O-5v"
- board text removed: "Limit Switch I/O-5v"
- board text removed: "Power out"
- board text removed: "Skrot AB SA6DGJ 2021-06-01 Elevation controll"
- board text removed: "UART RX - TX"
